Commit message: Changes to URDF files and adding sensor data with joint to xacro file

File: src/mars_rover/urdf/mars_rover.urdf (robot description, URDF)
Before this commit: robot mars_rover, 5 links, 4 joints
Links:
- added link gazebo_base_link
Joints:
- added joint gazebo_base_link: type None, parent gazebo_base_link, child base_link

File: src/mars_rover/urdf/mars_rover.urdf.xacro (robot description, xacro)
@@ -8,4 +8,40 @@
 	<xacro:include filename="${find mars_rover)/urdf/ylidar.urdf"/>
 <!-- Add your gazebo sensors here -->
+	<gazebo reference="base_laser">
+		<!-- <gravity>true</gravity> -->
+		<!-- Gazebo has fixed set of Sensors types. Check them out here <> -->
+		<sensor name="laser" type="ray">
+			<!-- Add in your sensor characteristics -->
+			<pose> 0 0 0 0 0 0 </pose>
+			<visualise>true</visualise>
+			<update_rate>40</update_rate>
+			<!-- <always_on>true</always_on> -->
+			<ray>
+				<scan>
+					<horizontal>
+						<samples>720</samples>
+						<resolution>1</resolution>
+						<min_angle>-1.570796</min_angle>
+              			<max_angle>1.570796</max_angle>
+              		</horizontal>
+              	</scan>
+              	<range>
+              		<min>0.10</min>
+              		<max>30.0</max>
+              		<resolution>0.01</resolution>
+              	</range>
+              	<noise>
+              		<type>gaussian</type>
+              		<mean>0.0</mean>
+              		<stddev>0.01</stddev>
+              	</noise>
+            </ray>
+            <plugin name="gazebo_ros_head_hokuyo_controller" filename="libgazebo_ros_laser.so">
+            	<!-- Use topic name as /my_robot/scan -->
+				<topicName></topicName>
+				<frameName>laser_frame</frameName>
+			</plugin>
+		</sensor>
+	</gazebo>
 <!--  Gazebo plugin for control here is already added for you -->
 	<gazebo>
@@ -17,3 +53,13 @@
 	</gazebo>
 <!-- Create a joint between your robot and sensor -->
+	<joint
+    name="base_laser_joint"
+    type="fixed">
+    <parent
+      link="base_link" />
+    <child
+      link="base_laser" />
+    <axis
+      xyz="0 0 0" />
+  </joint>
 </robot>

Commit message: Adding final urdf file for mar rover

File: src/mars_rover/urdf/mars_rover.urdf (robot description, URDF)
Before this commit: robot mars_rover, 6 links, 5 joints
Joints:
- joint gazebo_base_link: type None -> fixed

File: src/mars_rover/urdf/mars_rover.urdf.xacro (robot description, xacro)
@@ -5,6 +5,6 @@
 	<!-- Include Robot's urdf filepath -->
 	<!-- Include Lidar's urdf filepath -->
-	<xacro:include filename="${find mars_rover)/urdf/mars_rover.urdf"/>
-	<xacro:include filename="${find mars_rover)/urdf/ylidar.urdf"/>
+	<xacro:include filename="mars_rover.urdf"/>
+	<xacro:include filename="ydlidar.urdf"/>
 <!-- Add your gazebo sensors here -->
 	<gazebo reference="base_laser">
